Commit message: rearrange from C

File: robot_ws/src/buddy_description/urdf/arm_placeholder.urdf.xacro (robot description, xacro)
@@ -1,9 +1,9 @@
 <?xml version="1.0"?>
+<!-- PLACEHOLDER arm mount only. Replace with the selected arm model when chosen. -->
 <robot xmlns:xacro="http://www.ros.org/wiki/xacro">
   <xacro:macro name="buddy_arm_placeholder">
-    <!-- Placeholder only. Replace with selected arm package/model when known. -->
     <link name="arm_base_link">
-      <visual><geometry><box size="0.12 0.12 0.04"/></geometry></visual>
-      <collision><geometry><box size="0.12 0.12 0.04"/></geometry></collision>
+      <visual><geometry><box size="0.10 0.10 0.04"/></geometry></visual>
+      <collision><geometry><box size="0.10 0.10 0.04"/></geometry></collision>
       <inertial>
         <mass value="0.5"/>
@@ -14,5 +14,5 @@
       <parent link="base_link"/>
       <child link="arm_base_link"/>
-      <origin xyz="0.00 0 0.14" rpy="0 0 0"/>
+      <origin xyz="0.0 0 0.07" rpy="0 0 0"/>
     </joint>
   </xacro:macro>

File: robot_ws/src/buddy_description/urdf/base_four_wheel_diff.urdf.xacro (robot description, xacro)
@@ -1,4 +1,14 @@
 <?xml version="1.0"?>
 <robot xmlns:xacro="http://www.ros.org/wiki/xacro">
+  <!-- Solid-box inertia helper -->
+  <xacro:macro name="box_inertia" params="m x y z">
+    <inertial>
+      <mass value="${m}"/>
+      <inertia
+        ixx="${(1.0/12.0)*m*(y*y + z*z)}" ixy="0.0" ixz="0.0"
+        iyy="${(1.0/12.0)*m*(x*x + z*z)}" iyz="0.0"
+        izz="${(1.0/12.0)*m*(x*x + y*y)}"/>
+    </inertial>
+  </xacro:macro>
   <xacro:macro name="buddy_base">
     <link name="base_footprint"/>
@@ -6,19 +16,17 @@
       <parent link="base_footprint"/>
       <child link="base_link"/>
-      <origin xyz="0 0 0.10" rpy="0 0 0"/>
+      <origin xyz="0 0 ${base_center_z}" rpy="0 0 0"/>
     </joint>
     <link name="base_link">
       <visual>
         <geometry><box size="${base_length} ${base_width} ${base_height}"/></geometry>
+        <material name="body_gray"><color rgba="0.45 0.45 0.45 1"/></material>
       </visual>
       <collision>
         <geometry><box size="${base_length} ${base_width} ${base_height}"/></geometry>
       </collision>
-      <inertial>
-        <mass value="15.0"/>
-        <!-- Placeholder inertia. Replace after chassis/mass distribution are known. -->
-        <inertia ixx="0.30" ixy="0.0" ixz="0.0" iyy="0.45" iyz="0.0" izz="0.55"/>
-      </inertial>
+      <xacro:box_inertia m="${base_mass}" x="${base_length}" y="${base_width}" z="${base_height}"/>
     </link>
+    <!-- Wheel macro: cylinder about Y axis, inertia from wheel_mass/radius/width -->
     <xacro:macro name="wheel" params="name x y">
       <link name="${name}_link">
@@ -26,4 +34,5 @@
           <origin rpy="1.57079632679 0 0" xyz="0 0 0"/>
           <geometry><cylinder radius="${wheel_radius}" length="${wheel_width}"/></geometry>
+          <material name="wheel_black"><color rgba="0.02 0.02 0.02 1"/></material>
         </visual>
         <collision>
@@ -32,6 +41,9 @@
         </collision>
         <inertial>
-          <mass value="0.8"/>
-          <inertia ixx="0.003" ixy="0" ixz="0" iyy="0.003" iyz="0" izz="0.003"/>
+          <mass value="${wheel_mass}"/>
+          <inertia
+            ixx="${(1.0/12.0)*wheel_mass*(3.0*wheel_radius*wheel_radius + wheel_width*wheel_width)}" ixy="0" ixz="0"
+            iyy="${0.5*wheel_mass*wheel_radius*wheel_radius}" iyz="0"
+            izz="${(1.0/12.0)*wheel_mass*(3.0*wheel_radius*wheel_radius + wheel_width*wheel_width)}"/>
         </inertial>
       </link>
@@ -43,8 +55,8 @@
       </joint>
     </xacro:macro>
-    <xacro:wheel name="left_front_wheel" x="${wheel_x}" y="${wheel_y}"/>
-    <xacro:wheel name="left_rear_wheel" x="-${wheel_x}" y="${wheel_y}"/>
-    <xacro:wheel name="right_front_wheel" x="${wheel_x}" y="-${wheel_y}"/>
-    <xacro:wheel name="right_rear_wheel" x="-${wheel_x}" y="-${wheel_y}"/>
+    <xacro:wheel name="left_front_wheel"  x="${wheel_x}"  y="${wheel_y}"/>
+    <xacro:wheel name="left_rear_wheel"   x="${-wheel_x}" y="${wheel_y}"/>
+    <xacro:wheel name="right_front_wheel" x="${wheel_x}"  y="${-wheel_y}"/>
+    <xacro:wheel name="right_rear_wheel"  x="${-wheel_x}" y="${-wheel_y}"/>
   </xacro:macro>
 </robot>

File: robot_ws/src/buddy_description/urdf/buddy.urdf.xacro (robot description, xacro)
@@ -1,116 +1,26 @@
 <?xml version="1.0"?>
+<!-- THE single robot description entry point for Buddy v0.1.
+     RViz, Gazebo, and (optionally) ros2_control all build from this file.
+     Geometry lives in buddy_params.xacro. -->
 <robot xmlns:xacro="http://www.ros.org/wiki/xacro" name="buddy">
-  <!-- Minimal active model for RViz and early frame design. -->
-  <xacro:arg name="base_length" default="0.28"/>
-  <xacro:arg name="base_width" default="0.22"/>
-  <xacro:arg name="base_height" default="0.10"/>
-  <xacro:arg name="base_center_z" default="0.10"/>
-  <xacro:arg name="wheel_radius" default="0.06"/>
-  <xacro:arg name="wheel_width" default="0.035"/>
-  <xacro:arg name="wheel_x" default="0.09"/>
-  <xacro:arg name="wheel_y" default="0.13"/>
-  <xacro:arg name="wheel_z" default="-0.04"/>
-  <xacro:property name="base_length" value="$(arg base_length)"/>
-  <xacro:property name="base_width" value="$(arg base_width)"/>
-  <xacro:property name="base_height" value="$(arg base_height)"/>
-  <xacro:property name="base_center_z" value="$(arg base_center_z)"/>
-  <xacro:property name="wheel_radius" value="$(arg wheel_radius)"/>
-  <xacro:property name="wheel_width" value="$(arg wheel_width)"/>
-  <xacro:property name="wheel_x" value="$(arg wheel_x)"/>
-  <xacro:property name="wheel_y" value="$(arg wheel_y)"/>
-  <xacro:property name="wheel_z" value="$(arg wheel_z)"/>
-  <material name="body_gray"><color rgba="0.45 0.45 0.45 1"/></material>
-  <material name="wheel_black"><color rgba="0.02 0.02 0.02 1"/></material>
-  <material name="sensor_blue"><color rgba="0.1 0.2 0.8 1"/></material>
-  <material name="camera_green"><color rgba="0.0 0.5 0.2 1"/></material>
-  <link name="base_footprint"/>
-  <joint name="base_footprint_joint" type="fixed">
-    <parent link="base_footprint"/>
-    <child link="base_link"/>
-    <origin xyz="0 0 ${base_center_z}" rpy="0 0 0"/>
-  </joint>
-  <link name="base_link">
-    <visual>
-      <geometry><box size="${base_length} ${base_width} ${base_height}"/></geometry>
-      <material name="body_gray"/>
-    </visual>
-    <collision>
-      <geometry><box size="${base_length} ${base_width} ${base_height}"/></geometry>
-    </collision>
-    <inertial>
-      <mass value="20.0"/>
-      <inertia ixx="0.20" ixy="0" ixz="0" iyy="0.20" iyz="0" izz="0.25"/>
-    </inertial>
-  </link>
-  <xacro:macro name="wheel" params="name x y">
-    <link name="${name}_link">
-      <visual>
-        <origin xyz="0 0 0" rpy="1.57079632679 0 0"/>
-        <geometry><cylinder radius="${wheel_radius}" length="${wheel_width}"/></geometry>
-        <material name="wheel_black"/>
-      </visual>
-      <collision>
-        <origin xyz="0 0 0" rpy="1.57079632679 0 0"/>
-        <geometry><cylinder radius="${wheel_radius}" length="${wheel_width}"/></geometry>
-      </collision>
-      <inertial>
-        <mass value="0.50"/>
-        <inertia ixx="0.001" ixy="0" ixz="0" iyy="0.001" iyz="0" izz="0.001"/>
-      </inertial>
-    </link>
-    <joint name="${name}_joint" type="continuous">
-      <parent link="base_link"/>
-      <child link="${name}_link"/>
-      <origin xyz="${x} ${y} ${wheel_z}" rpy="0 0 0"/>
-      <axis xyz="0 1 0"/>
-    </joint>
-  </xacro:macro>
-  <xacro:wheel name="left_front_wheel"  x="${wheel_x}"  y="${wheel_y}"/>
-  <xacro:wheel name="left_rear_wheel"   x="-${wheel_x}" y="${wheel_y}"/>
-  <xacro:wheel name="right_front_wheel" x="${wheel_x}"  y="-${wheel_y}"/>
-  <xacro:wheel name="right_rear_wheel"  x="-${wheel_x}" y="-${wheel_y}"/>
-  <link name="base_laser">
-    <visual>
-      <geometry><cylinder radius="0.035" length="0.035"/></geometry>
-      <material name="sensor_blue"/>
-    </visual>
-  </link>
-  <joint name="base_laser_joint" type="fixed">
-    <parent link="base_link"/>
-    <child link="base_laser"/>
-    <origin xyz="0.06 0 0.10" rpy="0 0 0"/>
-  </joint>
-  <link name="front_camera_link">
-    <visual>
-      <geometry><box size="0.07 0.025 0.025"/></geometry>
-      <material name="camera_green"/>
-    </visual>
-  </link>
-  <joint name="front_camera_joint" type="fixed">
-    <parent link="base_link"/>
-    <child link="front_camera_link"/>
-    <origin xyz="0.15 0 0.06" rpy="0 0 0"/>
-  </joint>
-  <link name="front_camera_optical_frame"/>
-  <joint name="front_camera_optical_joint" type="fixed">
-    <parent link="front_camera_link"/>
-    <child link="front_camera_optical_frame"/>
-    <origin xyz="0 0 0" rpy="-1.57079632679 0 -1.57079632679"/>
-  </joint>
-  <link name="imu_link">
-    <visual><geometry><box size="0.035 0.025 0.010"/></geometry></visual>
-  </link>
-  <joint name="imu_joint" type="fixed">
-    <parent link="base_link"/>
-    <child link="imu_link"/>
-    <origin xyz="0 0 0.055" rpy="0 0 0"/>
-  </joint>
-  <link name="arm_base_placeholder_link">
-    <visual><geometry><box size="0.08 0.08 0.025"/></geometry></visual>
-  </link>
-  <joint name="arm_base_placeholder_joint" type="fixed">
-    <parent link="base_link"/>
-    <child link="arm_base_placeholder_link"/>
-    <origin xyz="0 0 0.075" rpy="0 0 0"/>
-  </joint>
+  <!-- Build switches -->
+  <xacro:arg name="use_gazebo" default="true"/>       <!-- emit gz plugins + sensors -->
+  <xacro:arg name="use_ros2_control" default="false"/> <!-- emit ros2_control (real hardware) -->
+  <xacro:property name="use_gazebo" value="$(arg use_gazebo)"/>
+  <xacro:property name="use_ros2_control" value="$(arg use_ros2_control)"/>
+  <xacro:include filename="$(find buddy_description)/urdf/buddy_params.xacro"/>
+  <xacro:include filename="$(find buddy_description)/urdf/base_four_wheel_diff.urdf.xacro"/>
+  <xacro:include filename="$(find buddy_description)/urdf/sensors_rgbd_2d_lidar.urdf.xacro"/>
+  <xacro:include filename="$(find buddy_description)/urdf/arm_placeholder.urdf.xacro"/>
+  <xacro:include filename="$(find buddy_description)/urdf/buddy.gazebo.xacro"/>
+  <xacro:include filename="$(find buddy_description)/urdf/ros2_control_four_wheel_base.xacro"/>
+  <xacro:buddy_base/>
+  <xacro:buddy_sensors/>
+  <xacro:buddy_arm_placeholder/>
+  <xacro:if value="${use_gazebo}">
+    <xacro:buddy_gazebo/>
+  </xacro:if>
+  <xacro:if value="${use_ros2_control}">
+    <xacro:buddy_ros2_control/>
+  </xacro:if>
 </robot>

File: robot_ws/src/buddy_description/urdf/sensors_rgbd_2d_lidar.urdf.xacro (robot description, xacro)
@@ -2,21 +2,27 @@
 <robot xmlns:xacro="http://www.ros.org/wiki/xacro">
   <xacro:macro name="buddy_sensors">
+    <!-- 2D LiDAR on a short mast above the body. -->
     <link name="base_laser">
-      <visual><geometry><cylinder radius="0.04" length="0.04"/></geometry></visual>
+      <visual>
+        <geometry><cylinder radius="0.035" length="0.035"/></geometry>
+        <material name="sensor_blue"><color rgba="0.1 0.2 0.8 1"/></material>
+      </visual>
     </link>
     <joint name="base_laser_joint" type="fixed">
       <parent link="base_link"/>
       <child link="base_laser"/>
-      <!-- Update after LiDAR mount is designed. -->
-      <origin xyz="0.18 0 0.16" rpy="0 0 0"/>
+      <origin xyz="0.06 0 0.10" rpy="0 0 0"/>
     </joint>
+    <!-- RGB-D camera near the front face. -->
     <link name="front_camera_link">
-      <visual><geometry><box size="0.09 0.03 0.03"/></geometry></visual>
+      <visual>
+        <geometry><box size="0.07 0.025 0.025"/></geometry>
+        <material name="camera_green"><color rgba="0.0 0.5 0.2 1"/></material>
+      </visual>
     </link>
     <joint name="front_camera_joint" type="fixed">
       <parent link="base_link"/>
       <child link="front_camera_link"/>
-      <!-- Update pitch/height after camera model and task-space are known. -->
-      <origin xyz="0.28 0 0.14" rpy="0 0 0"/>
+      <origin xyz="0.13 0 0.02" rpy="0 0 0"/>
     </joint>
     <link name="front_camera_optical_frame"/>
@@ -24,14 +30,14 @@
       <parent link="front_camera_link"/>
       <child link="front_camera_optical_frame"/>
-      <!-- Optical frame convention: z forward, x right, y down. -->
+      <!-- Optical convention: z forward, x right, y down. -->
       <origin xyz="0 0 0" rpy="-1.57079632679 0 -1.57079632679"/>
     </joint>
     <link name="imu_link">
-      <visual><geometry><box size="0.04 0.03 0.01"/></geometry></visual>
+      <visual><geometry><box size="0.03 0.02 0.01"/></geometry></visual>
     </link>
     <joint name="imu_joint" type="fixed">
       <parent link="base_link"/>
       <child link="imu_link"/>
-      <origin xyz="0 0 0.11" rpy="0 0 0"/>
+      <origin xyz="0 0 0.0" rpy="0 0 0"/>
     </joint>
   </xacro:macro>
