Commit message: Select wheels: 96mm goBILDA Hogback (ADR-0004), amend clearance requirement
The 0.06 m wheel radius used in motor sizing was an unsourced URDF
placeholder. goBILDA traction wheels top out at 96 mm; the Hogback's
crowned tread is purpose-designed to reduce skid-steer pivot scrub —
Buddy's dominant torque load case.

Decision: 4x Hogback 96 mm (50A, $9.99 ea) + 4x 8 mm REX-bore hubs,
~$76 all-in. Trade: ground-clearance requirement amended 0.05 -> 0.038 m
(the 0.05 was a round-number guess; indoor thresholds are 5-20 mm).

At r = 0.048 m the envelope relaxes everywhere it was tight:
design case 1.47 -> 1.18 N·m @ 149 RPM; pivot band 2.9-3.8 -> 2.29-3.06,
giving the selected motor 22% stall margin at mu = 0.8 (was marginal).

Cascade applied:
- requirements yaml: ground_clearance_m 0.038 with amendment note
- buddy_params.xacro: wheel_radius 0.048, wheel_mass 0.2, base_center_z
  0.10 -> 0.088 (axle height must equal wheel radius or sim wheels float)
- torque envelope figure + sweep CSV regenerated; figure title now
  derives from parameters instead of hardcoding the radius
- derivation doc substitutions redone at r = 0.048; noted the crowned
  tread as model conservatism
- sizing doc envelope/targets updated; M01 gains a dated postscript
  (historical numbers preserved, figure caption matches current figure)
- ADR-0004 records the decision and the requirement amendment

Co-Authored-By: Claude Fable 5 <noreply@anthropic.com>

File: robot_ws/src/buddy_description/urdf/buddy_params.xacro (robot description, xacro)
@@ -14,10 +14,14 @@
   <xacro:property name="base_height" value="0.10"/>
   <xacro:property name="base_mass"   value="18.0"/>
-  <!-- base_link center height above ground (base_footprint -> base_link) -->
-  <xacro:property name="base_center_z" value="0.10"/>
-  <!-- Wheels -->
-  <xacro:property name="wheel_radius" value="0.06"/>
+  <!-- base_link center height above ground (base_footprint -> base_link).
+       Constraint: base_center_z + wheel_z must equal wheel_radius (axle height),
+       or the wheels float/sink in sim. 0.088 - 0.04 = 0.048 ✓.
+       Ground clearance = base_center_z - base_height/2 = 0.038 m (ADR-0004). -->
+  <xacro:property name="base_center_z" value="0.088"/>
+  <!-- Wheels: goBILDA Hogback traction wheel, 96mm dia, 50A (ADR-0004).
+       Width and mass are nominal — verify by measurement on receipt. -->
+  <xacro:property name="wheel_radius" value="0.048"/>
   <xacro:property name="wheel_width"  value="0.035"/>
-  <xacro:property name="wheel_mass"   value="0.8"/>
+  <xacro:property name="wheel_mass"   value="0.2"/>
   <xacro:property name="wheel_x"      value="0.09"/>   <!-- +/- from center, fore/aft -->
   <xacro:property name="wheel_y"      value="0.13"/>   <!-- +/- from center, left/right (track/2) -->

Commit message: Add parametric build: one yaml drives derivations, figures, URDF, and CSV
Design values previously lived in five hand-synced places (requirements
yaml, buddy_params.xacro, torque_sweep CLI defaults, figure-script
constants, and markdown prose). The wheel change proved the failure mode:
every substitution had to be chased by hand, and a rounding error
(3.06 vs computed 3.05 N·m) had already crept into three docs.

Single source of truth, split by responsibility:
- design_params.yaml — chosen/assumed values (geometry, motor/wheel
  specs, crr/mu/eta/SF); requirements yaml keeps requirements; no overlap.
- buddy_calcs/ — loader + drive equations; every consumer imports it
  (figure scripts, torque_sweep CLI, notebooks, xacro generator).

python3 tools/build.py regenerates, deterministically (byte-identical
consecutive builds):
- buddy_params.xacro — now a GENERATED file with a do-not-edit header;
  base_center_z derived so axle height always equals wheel radius.
- docs/analysis/drive_torque_and_pivot_scrub.md — exported from the new
  marimo notebook (.py, same basename), where every substituted number
  is computed; explore live with `marimo edit`.
- both figures (parametrized; FBD wheels were still drawn at the stale
  120 mm — parametrization fixed that automatically) and the sweep CSV.
- Validation gate: derived ground clearance is checked against the
  requirements yaml before anything regenerates.

Verified end-to-end: SF 2.0 -> 1.5 propagated 1.18 -> 0.88 N·m through
the derivation, figure legend, design-point annotation, and CSV in one
build; reverted cleanly. Docs updated to the new source-of-truth story
(PROJECT_CONTEXT, README, SIMULATION_START_HERE, sizing doc, portfolio
README); rounding drift fixed to the computed 3.05 N·m.

Co-Authored-By: Claude Fable 5 <noreply@anthropic.com>

File: robot_ws/src/buddy_description/urdf/buddy_params.xacro (robot description, xacro)
@@ -1,24 +1,23 @@
 <?xml version="1.0"?>
-<!-- SINGLE SOURCE OF TRUTH for Buddy geometry and mass.
-     Every other xacro (base, sensors, gazebo) reads these properties.
-     Change a number here and it propagates to RViz, Gazebo physics, and the
-     diff-drive plugin at once.
-     NOTE (placeholder warning): the current 0.28 x 0.22 x 0.10 m body at ~30 kg
-     gross is physically dense and almost certainly too small for the real robot.
-     It is kept only because the live sim and torque defaults already used it.
-     Revisit once chassis dimensions are chosen, then this is the only file to edit. -->
+<!-- ============================ GENERATED FILE ============================
+     DO NOT EDIT. Generated by tools/build.py from design_params.yaml — edit
+     that file and re-run `python3 tools/build.py`. Values here feed RViz,
+     Gazebo physics, and the diff-drive plugin at once.
+     NOTE (placeholder warning): the chassis box is a placeholder and almost
+     certainly not the final shape. Revisit with chassis CAD — in
+     design_params.yaml, never here.
+     ======================================================================= -->
 <robot xmlns:xacro="http://www.ros.org/wiki/xacro">
   <!-- Body box -->
   <xacro:property name="base_length" value="0.28"/>
   <xacro:property name="base_width"  value="0.22"/>
-  <xacro:property name="base_height" value="0.10"/>
-  <xacro:property name="base_mass"   value="18.0"/>
+  <xacro:property name="base_height" value="0.1"/>
+  <xacro:property name="base_mass"   value="18"/>
   <!-- base_link center height above ground (base_footprint -> base_link).
-       Constraint: base_center_z + wheel_z must equal wheel_radius (axle height),
-       or the wheels float/sink in sim. 0.088 - 0.04 = 0.048 ✓.
-       Ground clearance = base_center_z - base_height/2 = 0.038 m (ADR-0004). -->
+       DERIVED as wheel_radius - wheel_z so axle height always equals wheel
+       radius (wheels touch ground in sim). Ground clearance
+       = base_center_z - base_height/2 = 0.038 m. -->
   <xacro:property name="base_center_z" value="0.088"/>
-  <!-- Wheels: goBILDA Hogback traction wheel, 96mm dia, 50A (ADR-0004).
-       Width and mass are nominal — verify by measurement on receipt. -->
+  <!-- Wheels: goBILDA 3626-0014-0096 Hogback (96 mm, 50A) -->
   <xacro:property name="wheel_radius" value="0.048"/>
   <xacro:property name="wheel_width"  value="0.035"/>
