Commit message: Define the chassis CAD interface, and a slot for measured inertia
The chassis is the first part designed in CAD rather than in design_params.yaml,
which creates a risk the rest of the repo does not have: two sources of truth for
the same number - the YAML the URDF, Gazebo and the torque envelope believe,
versus the model actually built. When those drift nothing errors; the simulation
just describes a robot that does not exist. Same failure class as the Mermaid
diagram deleted on 07-28 and the 0.08 m wheel radius in the deleted CAN stubs.

chassis_interface.md draws the line. The YAML keeps owning anything the URDF,
torque analysis, power model or a requirement consumes - track, wheelbase, wheel
radius, bounding box, ground clearance - and CAD must satisfy those rather than
choose them. CAD owns ribs, fillets, bosses, routing, print orientation, none of
which belong in the YAML. Three properties flow back the other way: mass, centre
of mass, inertia tensor, read from SolidWorks mass properties and typed in. The
build never parses a CAD file.

Adds the fields and wires them through. While com_m and inertia_kgm2 are null the
URDF keeps its uniform solid-box approximation; fill both and it switches to the
real tensor with a proper inertial origin. Verified all three paths on the
Jetson with xacro: placeholder branch emits box inertia and no origin, measured
branch emits the CoM offset and products of inertia, and a partially filled
tensor is refused rather than silently zeroed.

The CoM matters more than the mass here. The 20 degree ramp requirement is a
tipping problem, and the box approximation assumes the centre of mass sits at the
geometric centre - wrong the moment a 2.1 kg pack goes anywhere else. Until com_m
is filled the sim cannot say anything trustworthy about tipping.

Co-Authored-By: Claude Opus 5 <noreply@anthropic.com>

File: robot_ws/src/buddy_description/urdf/base_four_wheel_diff.urdf.xacro (robot description, xacro)
@@ -26,5 +26,18 @@
         <geometry><box size="${base_length} ${base_width} ${base_height}"/></geometry>
       </collision>
-      <xacro:box_inertia m="${base_mass}" x="${base_length}" y="${base_width}" z="${base_height}"/>
+      <!-- Inertia: measured from CAD when available, else the solid-box
+           approximation. Both branches come from design_params.yaml via the
+           generated buddy_params.xacro — see docs/system_model/chassis_interface.md -->
+      <xacro:unless value="${measured_inertia}">
+        <xacro:box_inertia m="${base_mass}" x="${base_length}" y="${base_width}" z="${base_height}"/>
+      </xacro:unless>
+      <xacro:if value="${measured_inertia}">
+        <inertial>
+          <origin xyz="${com_x} ${com_y} ${com_z}" rpy="0 0 0"/>
+          <mass value="${base_mass}"/>
+          <inertia ixx="${base_ixx}" ixy="${base_ixy}" ixz="${base_ixz}"
+                   iyy="${base_iyy}" iyz="${base_iyz}" izz="${base_izz}"/>
+        </inertial>
+      </xacro:if>
     </link>
     <!-- Wheel macro: cylinder about Y axis, inertia from wheel_mass/radius/width -->

File: robot_ws/src/buddy_description/urdf/buddy_params.xacro (robot description, xacro)
@@ -14,4 +14,21 @@
   <xacro:property name="base_height" value="0.1"/>
   <xacro:property name="base_mass"   value="18"/>
+  <!-- Inertial provenance: "placeholder".
+       measured_inertia=false -> the URDF derives a uniform solid-box inertia
+       about the geometric centre (the long-standing placeholder behaviour).
+       Fill chassis.com_m and chassis.inertia_kgm2 in design_params.yaml from
+       SolidWorks mass properties and this flips to true, so the sim inherits
+       the real mass distribution — which is what the 20 deg ramp tipping case
+       actually depends on. See docs/system_model/chassis_interface.md -->
+  <xacro:property name="measured_inertia" value="false"/>
+  <xacro:property name="com_x" value="0"/>
+  <xacro:property name="com_y" value="0"/>
+  <xacro:property name="com_z" value="0"/>
+  <xacro:property name="base_ixx" value="0"/>
+  <xacro:property name="base_iyy" value="0"/>
+  <xacro:property name="base_izz" value="0"/>
+  <xacro:property name="base_ixy" value="0"/>
+  <xacro:property name="base_ixz" value="0"/>
+  <xacro:property name="base_iyz" value="0"/>
   <!-- base_link center height above ground (base_footprint -> base_link).
        DERIVED as wheel_radius - wheel_z so axle height always equals wheel
