File: electronics/KiCAD/system_wiring/system_wiring.kicad_sch (KiCad schematic)
At the start: 13 parts, among them K1 E-stop contactor ~40A, U1 NUCLEO-G474RE (JP3 = E5V), U10 12V buck >=5A (Jetson), U11 5V buck >=3A (logic)

Commit message: Change the bus to 4S LiFePO4 (ADR-0005 amendment 2)
Compiling sourced options for the unbought parts found two problems that made
the specified power architecture unbuildable.

The Jetson 12 V rail could not exist. A step-down needs input above output, and
a 3S bus is 12.6 V only at full charge, bottoming at 9.0 V. The named example
part (D24V50F12) does not appear to exist either - Pololu fixed 12 V step-downs
are 500 mA and the 5 A D24V50F5 is a 5 V part. That part number had been carried
in the plan for three weeks.

The >=50 A BMS was not purchasable in 3S. Stock 12 V Li-ion packs ship 10-30 A
boards against a 46 A designed peak - a pack that trips on the first carpet
pivot, which is what the shopping list already warned about.

LiFePO4 answers both: 10.0-14.6 V sits inside the dev kit 9-20 V window with
margin at both ends, so the Jetson feeds straight off the bus and the converter
is deleted rather than re-specified, and a 100 A BMS is the default in that
category. Recomputed, not asserted: system current 4.95 -> 4.30 A, designed peak
37.0 -> 36.3 A, peak incl. arms 47.0 -> 46.3 A, capacity >=14 -> >=12.1 Ah,
torque at the 8 A limit unchanged at 3.23 N.m since torque per amp is voltage
independent. BMS >=50 A and the 60 A fuse both stand; validate() passes.

Costs recorded rather than buried: ~+1.3 kg, larger than the +0.6-0.8 kg the
07-14 amendment absorbed, and motors running above their 12 V nominal. The mass
is the real one and chassis CAD settles it.

Renames the ADR file, which asserted a chemistry it no longer chooses.

Co-Authored-By: Claude Opus 5 <noreply@anthropic.com>
Parts:
- BT1: value 3S Li-ion + BMS >= 50A (9-12.6V) -> 3S Li-ion + BMS >= 50A (10-14.6V)
Changed lines of the file:
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@@
     (exclude_from_sim no) (in_bom yes) (on_board yes) (dnp no)
     (property "Reference" "BT1" (at 54.61 76.17 0) (effects (font (size 1.27 1.27))))
-    (property "Value" "3S Li-ion + BMS >= 50A (9-12.6V)" (at 54.61 114.33 0) (effects (font (size 1.27 1.27))))
+    (property "Value" "3S Li-ion + BMS >= 50A (10-14.6V)" (at 54.61 114.33 0) (effects (font (size 1.27 1.27))))
     (pin "1")
     (pin "2")
